File: PMIC.sch (KiCad schematic (older format))
At the start: 60 parts, among them U3 BD71847MWV, Y1 Crystal

Commit message: Corrections for bom of v0.1
Parts:
- C69, C70: Part GRM0335C1H180JA01D -> GCM1555C1H180JA16D; Vendorpart 490-6117-1-ND -> 490-12650-1-ND
Changed lines of the file:
@@
 F 3 "~" H 3350 8450 50  0001 C CNN
 F 4 "Murata" H 3350 8450 50  0001 C CNN "Mfgr"
-F 5 "GRM0335C1H180JA01D" H 3350 8450 50  0001 C CNN "Part"
-F 6 "490-6117-1-ND" H 3350 8450 50  0001 C CNN "Vendorpart"
+F 5 "GCM1555C1H180JA16D" H 3350 8450 50  0001 C CNN "Part"
+F 6 "490-12650-1-ND" H 3350 8450 50  0001 C CNN "Vendorpart"
 	1    3350 8450
 	-1   0    0    1
@@
 F 3 "~" H 4200 8450 50  0001 C CNN
 F 4 "Murata" H 4200 8450 50  0001 C CNN "Mfgr"
-F 5 "GRM0335C1H180JA01D" H 4200 8450 50  0001 C CNN "Part"
-F 6 "490-6117-1-ND" H 4200 8450 50  0001 C CNN "Vendorpart"
+F 5 "GCM1555C1H180JA16D" H 4200 8450 50  0001 C CNN "Part"
+F 6 "490-12650-1-ND" H 4200 8450 50  0001 C CNN "Vendorpart"
 	1    4200 8450
 	-1   0    0    1
