File: USB.sch (KiCad schematic (older format))
At the start: 53 parts, among them J1 USB_C_Receptacle, J7 USB_MICRO_B, U1 IMX8MM, U11 AP2411SN-7, U2 CYPD4155-96BZXI, U6 SN65DSI86ZQER, U9 NX20P3483UK

Commit message: wip
Parts:
- removed C159, C160, C161, C163, C179, C192: 1uF, Capacitor_SMD:C_0201_0603Metric, symbol Device:C
- removed C162, C164, C165, C178, C180, C181, C182, C183, C184, C185, C186, C187, C188, C190, C191, C193: 0.1uF, Capacitor_SMD:C_0201_0603Metric, symbol Device:C
- removed R33: 11K, Resistor_SMD:R_0201_0603Metric, symbol Device:R
- removed R34: 1K, Resistor_SMD:R_0201_0603Metric, symbol Device:R
- removed R49: 4.7K, Resistor_SMD:R_0201_0603Metric, symbol Device:R
- removed R61: 51K, Resistor_SMD:R_0201_0603Metric, symbol Device:R
- removed U2: CYPD4155-96BZXI, mxenc:BGA-121_11x11_6.0x6.0mm, symbol mxenc:CYPD4155-96BZXI
- removed U6: SN65DSI86ZQER, mxenc:BGA64C50P9X9_500X500X100, symbol mxenc:SN65DSI86ZQER
Connections:
- net labels removed: AUXN, AUXP, DP_EN, DP_IRQ, DP_SCL, DP_SDA, DP_SUSP, DSI_CLK_N, DSI_CLK_P, DSI_D0_N, DSI_D0_P, DSI_D1_N, DSI_D1_P, DSI_D2_N, DSI_D2_P, DSI_D3_N, DSI_D3_P, HPD, HPD_H, ML0N, ML0P, ML1N, ML1P, ML2N, ML2P, ML3N, ML3P, USB2_SCL, USB2_SDA, VDD_1V8, VDD_PHY_1V2
- wire segments 285 -> 153
- no-connect marks 49 -> 2
Other:
- note removed: "1.8V"
- note removed: "3.3 V"
- note removed: "Configuration for 1080p60\n\nGPIO4:2 <=\n 3’b011\nDACP/N CLOCK FREQUENCY\n (DPPLL_CLK_SRC = 1) <=\n 486 MHz (DSIACLK / 18 = 27 MHz)\nREFCLK_FREQ <=\n 0x3"

Commit message: wip more new layout
Parts:
- removed D5, D6: D_TVS, Diode_SMD:D_0201_0603Metric, symbol Device:D_TVS
- removed J7: USB_MICRO_B, Connector_USB:USB_Micro-B_Molex_47346-0001, symbol Connector:USB_B_Micro
- removed unit 4 of U1
- removed U11: AP2411SN-7, Package_DFN_QFN:DFN-6-1EP_2x2mm_P0.65mm_EP1x1.6mm, symbol mxenc:AP2511SN-7
- added U2: PTN5110NHQZ, mxenc:HX2QFN-16_EP_2.85x2.85_Pitch0.4mm, symbol mxenc:PTN5110NHQZ
- J1: footprint mxenc:USBC_DX07S024JJ2R1300 -> mxenc:GCT_USB4110-GF-A; symbol Connector:USB_C_Receptacle -> Connector:USB_C_Receptacle_USB2.0
Connections:
- net GND: no longer J1.G (GND)
- net USB1_DN: now also J1.A7 (D-), J1.B7 (D-)
- net USB1_DP: now also J1.A6 (D+), J1.B6 (D+)
- net USB1_VBUS: now also F1.1, J1.A4 (VBUS), J1.A9 (VBUS), J1.B4 (VBUS), J1.B9 (VBUS)
- net USB2_DN: no longer J1.A7 (D-), J1.B7 (D-)
- net USB2_DP: no longer J1.A6 (D+), J1.B6 (D+)
- net USB2_VBUS: no longer F1.1, J1.A4 (VBUS), J1.A9 (VBUS), J1.B4 (VBUS), J1.B9 (VBUS)
- net USB2_PWR_SCL renamed USB1_PWR_SCL
- net USB2_PWR_SDA renamed USB1_PWR_SDA
- net USB2_VBUS_F renamed USB1_VBUS_F
- net USB2_VBUS_IN renamed USB1_VBUS_IN
- removed net USBC_RX1N: J1.B10 (RX1-)
- removed net USBC_RX1P: J1.B11 (RX1+)
- removed net USBC_RX2N: J1.A10 (RX2-)
- removed net USBC_RX2P: J1.A11 (RX2+)
- removed net USBC_TX1N: J1.A3 (TX1-)
- removed net USBC_TX1P: J1.A2 (TX1+)
- removed net USBC_TX2N: J1.B3 (TX2-)
- removed net USBC_TX2P: J1.B2 (TX2+)
- no-connect marks 2 -> 1
Other:
- note added: "47uF vs 100uF electrolytic?\n0.1uF already on input"
- note added: "have 1uF, 10uF, 100uF on VDD 5V pmic out"
- moved on the sheet: D3, D4
