File: USB.sch (KiCad schematic (older format))
At the start: 27 parts, among them J1 USB_C_Receptacle, U1 IMX8MM, U2 NX20P3483UK, U6 PTN5110NHQZ

Commit message: Cleanup remaining DRC problems from schematic
Parts:
- added C174, C175: 0.22uF, Capacitor_SMD:C_0201_0603Metric, symbol Device:C
- added R69, R70: 30K, Resistor_SMD:R_0201_0603Metric, symbol Device:R
Connections:
- net GND: now also C174.2, C175.2
- net USB1_VBUS: now also C175.1, R69.2; no longer U1.F22 (USB1_VBUS)
- net USB2_VBUS: now also C174.1, R70.2; no longer U1.F23 (USB2_VBUS)
- net USB1_ID: no longer names the net of U1.D22 (USB1_ID)
- new net USB1_VBUS_LV: R69.1, U1.F22 (USB1_VBUS)
- new net USB2_VBUS_LV: R70.1, U1.F23 (USB2_VBUS)
- no-connect marks 2 -> 3
Other:
- note added: "USB*_VBUS inputs operate at 3.3v"
- moved on the sheet: R33
Changed lines of the file:
@@
 $EndComp
-Wire Wire Line
-	3750 3550 3800 3550
-Wire Wire Line
-	3800 3650 3750 3650
 Wire Wire Line
 	3750 3800 3800 3800
-Text Label 3750 2950 0    50   ~ 0
+Text Label 3800 2950 0    50   ~ 0
 USB1_DP
-Text Label 3750 2850 0    50   ~ 0
+Text Label 3800 2850 0    50   ~ 0
 USB1_DN
-Text Label 3750 3100 0    50   ~ 0
-USB1_ID
 Wire Wire Line
 	13900 7700 13950 7700
@@
 Text Label 3800 3800 0    50   ~ 0
 USB2_ID
-Text Label 3800 3650 0    50   ~ 0
-USB2_DP
-Text Label 3800 3550 0    50   ~ 0
-USB2_DN
 $Comp
 L mxenc:NX20P3483UK U2
@@
 L Device:R R33
 U 1 1 5DBFE2FB
-P 4300 3500
-F 0 "R33" H 4370 3546 50  0000 L CNN
-F 1 "200" H 4370 3455 50  0000 L CNN
-F 2 "Resistor_SMD:R_0201_0603Metric" V 4230 3500 50  0001 C CNN
-F 3 "~" H 4300 3500 50  0001 C CNN
-F 4 "Yageo" H 4300 3500 50  0001 C CNN "Mfgr"
-F 5 "RC0201FR-07200RL" H 4300 3500 50  0001 C CNN "Part"
-F 6 "YAG2495CT-ND" H 4300 3500 50  0001 C CNN "Vendorpart"
-	1    4300 3500
-	1    0    0    -1
-$EndComp
-Wire Wire Line
-	3750 3250 4300 3250
-Wire Wire Line
-	4300 3250 4300 3350
+P 4450 3500
+F 0 "R33" H 4520 3546 50  0000 L CNN
+F 1 "200" H 4520 3455 50  0000 L CNN
+F 2 "Resistor_SMD:R_0201_0603Metric" V 4380 3500 50  0001 C CNN
+F 3 "~" H 4450 3500 50  0001 C CNN
+F 4 "Yageo" H 4450 3500 50  0001 C CNN "Mfgr"
+F 5 "RC0201FR-07200RL" H 4450 3500 50  0001 C CNN "Part"
+F 6 "YAG2495CT-ND" H 4450 3500 50  0001 C CNN "Vendorpart"
+	1    4450 3500
+	1    0    0    -1
+$EndComp
+Wire Wire Line
+	3750 3250 4450 3250
+Wire Wire Line
+	4450 3250 4450 3350
 $Comp
 L power:GND #PWR0213
 U 1 1 5DC0F263
-P 4300 3750
-F 0 "#PWR0213" H 4300 3500 50  0001 C CNN
-F 1 "GND" H 4305 3577 50  0000 C CNN
-F 2 "" H 4300 3750 50  0001 C CNN
-F 3 "" H 4300 3750 50  0001 C CNN
-	1    4300 3750
-	1    0    0    -1
-$EndComp
-Wire Wire Line
-	4300 3750 4300 3650
-Text Label 3950 2650 0    50   ~ 0
+P 4450 3750
+F 0 "#PWR0213" H 4450 3500 50  0001 C CNN
+F 1 "GND" H 4455 3577 50  0000 C CNN
+F 2 "" H 4450 3750 50  0001 C CNN
+F 3 "" H 4450 3750 50  0001 C CNN
+	1    4450 3750
+	1    0    0    -1
+$EndComp
+Wire Wire Line
+	4450 3750 4450 3650
+Text Label 6550 2350 0    50   ~ 0
 USB1_VBUS
-Wire Wire Line
-	3950 2650 3950 2750
-Wire Wire Line
-	3950 2750 3750 2750
-Text Label 3950 3350 0    50   ~ 0
+Text Label 6550 2650 0    50   ~ 0
 USB2_VBUS
-Wire Wire Line
-	3950 3350 3950 3450
-Wire Wire Line
-	3950 3450 3750 3450
 Text HLabel 9700 3950 0    50   BiDi ~ 0
 USB1_PWR_SDA
@@
 Text Notes 11500 2750 0    50   ~ 0
 have 1uF, 10uF, 100uF on VDD 5V pmic out
-Text Label 5500 3850 2    50   ~ 0
+Text Label 6100 4300 2    50   ~ 0
 USB2_VBUS
-Text Label 5500 3750 2    50   ~ 0
+Text Label 6100 4200 2    50   ~ 0
 USB2_DN
-Text Label 5500 3650 2    50   ~ 0
+Text Label 6100 4100 2    50   ~ 0
 USB2_DP
-Text Label 5500 3550 2    50   ~ 0
+Text Label 6100 4000 2    50   ~ 0
 USB2_ID
-Text GLabel 5500 3850 2    50   Input ~ 0
+Text GLabel 6100 4300 2    50   Input ~ 0
 USB2_VBUS
-Text GLabel 5500 3750 2    50   Input ~ 0
+Text GLabel 6100 4200 2    50   Input ~ 0
 USB2_DN
-Text GLabel 5500 3650 2    50   Input ~ 0
+Text GLabel 6100 4100 2    50   Input ~ 0
 USB2_DP
-Text GLabel 5500 3550 2    50   Input ~ 0
+Text GLabel 6100 4000 2    50   Input ~ 0
 USB2_ID
 $Comp
@@
 	1    0    0    -1
 $EndComp
+NoConn ~ 3750 3100
+Text Label 3800 2750 0    50   ~ 0
+USB1_VBUS_LV
+Text Label 5550 2350 2    50   ~ 0
+USB1_VBUS_LV
+Text Label 5550 2650 2    50   ~ 0
+USB2_VBUS_LV
+$Comp
+L Device:R R?
+U 1 1 5E8A7C7D
+P 5800 2350
+AR Path="/5E8A7C7D" Ref="R?"  Part="1"
+AR Path="/5D6742B7/5E8A7C7D" Ref="R69"  Part="1"
+F 0 "R69" V 5593 2350 50  0000 C CNN
+F 1 "30K" V 5684 2350 50  0000 C CNN
+F 2 "Resistor_SMD:R_0201_0603Metric" V 5730 2350 50  0001 C CNN
+F 3 "~" H 5800 2350 50  0001 C CNN
+F 4 "Yageo" H 5800 2350 50  0001 C CNN "Mfgr"
+F 5 "RC0201FR-0730KL" H 5800 2350 50  0001 C CNN "Part"
+F 6 "YAG2281CT-ND" H 5800 2350 50  0001 C CNN "Vendorpart"
+	1    5800 2350
+	0    -1   -1   0
+$EndComp
+Text Notes 5250 2150 0    50   ~ 0
+USB*_VBUS inputs operate at 3.3v
+$Comp
+L Device:R R?
+U 1 1 5E8BC0BD
+P 5800 2650
+AR Path="/5E8BC0BD" Ref="R?"  Part="1"
+AR Path="/5D6742B7/5E8BC0BD" Ref="R70"  Part="1"
+F 0 "R70" V 5593 2650 50  0000 C CNN
+F 1 "30K" V 5684 2650 50  0000 C CNN
+F 2 "Resistor_SMD:R_0201_0603Metric" V 5730 2650 50  0001 C CNN
+F 3 "~" H 5800 2650 50  0001 C CNN
+F 4 "Yageo" H 5800 2650 50  0001 C CNN "Mfgr"
+F 5 "RC0201FR-0730KL" H 5800 2650 50  0001 C CNN "Part"
+F 6 "YAG2281CT-ND" H 5800 2650 50  0001 C CNN "Vendorpart"
+	1    5800 2650
+	0    -1   -1   0
+$EndComp
+Wire Wire Line
+	5950 2350 6400 2350
+Wire Wire Line
+	5950 2650 6200 2650
+Wire Wire Line
+	6200 2650 6200 2750
+Connection ~ 6200 2650
+Wire Wire Line
+	6200 2650 6550 2650
+Wire Wire Line
+	6400 2350 6400 2750
+Connection ~ 6400 2350
+Wire Wire Line
+	6400 2350 6550 2350
+$Comp
+L power:GND #PWR0278
+U 1 1 5E9295BE
+P 6200 3050
+F 0 "#PWR0278" H 6200 2800 50  0001 C CNN
+F 1 "GND" H 6205 2877 50  0000 C CNN
+F 2 "" H 6200 3050 50  0001 C CNN
+F 3 "" H 6200 3050 50  0001 C CNN
+	1    6200 3050
+	1    0    0    -1
+$EndComp
+$Comp
+L power:GND #PWR0279
+U 1 1 5E929CCB
+P 6400 3050
+F 0 "#PWR0279" H 6400 2800 50  0001 C CNN
+F 1 "GND" H 6405 2877 50  0000 C CNN
+F 2 "" H 6400 3050 50  0001 C CNN
+F 3 "" H 6400 3050 50  0001 C CNN
+	1    6400 3050
+	1    0    0    -1
+$EndComp
+Wire Wire Line
+	3800 3650 3750 3650
+Text Label 3800 3650 0    50   ~ 0
+USB2_DP
+Wire Wire Line
+	3750 3550 3800 3550
+Text Label 3800 3550 0    50   ~ 0
+USB2_DN
+Wire Wire Line
+	3800 3450 3750 3450
+Text Label 3800 3450 0    50   ~ 0
+USB2_VBUS_LV
+Wire Wire Line
+	3800 2750 3750 2750
+Wire Wire Line
+	3750 2850 3800 2850
+Wire Wire Line
+	3800 2950 3750 2950
+Wire Wire Line
+	5550 2350 5650 2350
+Wire Wire Line
+	5550 2650 5650 2650
+$Comp
+L Device:C C?
+U 1 1 5EB3C320
+P 6200 2900
+AR Path="/5D1DA4BE/5EB3C320" Ref="C?"  Part="1"
+AR Path="/5D6742B7/5EB3C320" Ref="C174"  Part="1"
+F 0 "C174" H 5950 3000 50  0000 L CNN
+F 1 "0.22uF" H 5900 2800 50  0000 L CNN
+F 2 "Capacitor_SMD:C_0201_0603Metric" H 6238 2750 50  0001 C CNN
+F 3 "~" H 6200 2900 50  0001 C CNN
+F 4 "Murata" H 6200 2900 50  0001 C CNN "Mfgr"
+F 5 "GRM033C80J224KE90D" H 6200 2900 50  0001 C CNN "Part"
+F 6 "490-10392-1-ND" H 6200 2900 50  0001 C CNN "Vendorpart"
+	1    6200 2900
+	1    0    0    -1
+$EndComp
+$Comp
+L Device:C C?
+U 1 1 5EB4379E
+P 6400 2900
+AR Path="/5D1DA4BE/5EB4379E" Ref="C?"  Part="1"
+AR Path="/5D6742B7/5EB4379E" Ref="C175"  Part="1"
+F 0 "C175" H 6450 3000 50  0000 L CNN
+F 1 "0.22uF" H 6450 2800 50  0000 L CNN
+F 2 "Capacitor_SMD:C_0201_0603Metric" H 6438 2750 50  0001 C CNN
+F 3 "~" H 6400 2900 50  0001 C CNN
+F 4 "Murata" H 6400 2900 50  0001 C CNN "Mfgr"
+F 5 "GRM033C80J224KE90D" H 6400 2900 50  0001 C CNN "Part"
+F 6 "490-10392-1-ND" H 6400 2900 50  0001 C CNN "Vendorpart"
+	1    6400 2900
+	1    0    0    -1
+$EndComp

Commit message: Re-annotate schematics, add dnp field, and silkscreen cleanup
Parts:
- renumbered C93 to C162, C159 to C163, C160 to C164, C161 to C165, C174 to C166, C175 to C167, C164 to C168, C165 to C169, C168 to C170, C169 to C171, C170 to C172, C171 to C173, C172 to C174, D5 to D6, D6 to D7, D3 to D8, D4 to D9, J1 to J13, R69 to R64, R70 to R65, R33 to R66, R36 to R67, R37 to R68, R39 to R69, R34 to R70, U2 to U8, U6 to U9
