File: mxenc.sch (KiCad schematic (older format))
At the start: 29 parts, among them J4 Conn_01x06, J6 Conn_01x06, J8 Conn_01x06, SW1 SW_Push, SW2 SW_Push, U1 MIMX8MM6DVTLZAA, U10 24LC16, Y2 Crystal_GND24

Commit message: Tie boot0 to btn0 / sw1
Parts:
- removed JP1: SolderJumper_2_Open, Jumper:SolderJumper-2_P1.3mm_Open_RoundedPad1.0x1.5mm, symbol Jumper:SolderJumper_2_Open
- removed R53: 10K, Resistor_SMD:R_0201_0603Metric, symbol Device:R
Connections:
- wire segments 156 -> 151
Changed lines of the file:
@@
 $EndComp
-Wire Wire Line
-	6300 6200 6300 6250
-$Comp
-L mxenc:VDD_3V3 #PWR0243
-U 1 1 5D683A71
-P 6300 6200
-F 0 "#PWR0243" H 6300 6050 50  0001 C CNN
-F 1 "VDD_3V3" H 6315 6373 50  0000 C CNN
-F 2 "" H 6300 6200 50  0001 C CNN
-F 3 "" H 6300 6200 50  0001 C CNN
-	1    6300 6200
-	1    0    0    -1
-$EndComp
-Connection ~ 6000 7050
 Wire Wire Line
 	6000 7050 6000 7100
 Wire Wire Line
-	6300 7050 6000 7050
-Wire Wire Line
-	6300 7000 6300 7050
-Connection ~ 6300 6600
-Wire Wire Line
-	6300 6600 6300 6700
-Wire Wire Line
-	6300 6600 6300 6550
-Wire Wire Line
-	5700 6600 6300 6600
+	5700 6600 6000 6600
 Wire Wire Line
 	5700 6800 5700 6600
 Wire Wire Line
 	5100 6800 5700 6800
-$Comp
-L Jumper:SolderJumper_2_Open JP1
-U 1 1 5D620C66
-P 6300 6400
-F 0 "JP1" V 6254 6468 50  0000 L CNN
-F 1 "SolderJumper_2_Open" V 6345 6468 50  0000 L CNN
-F 2 "Jumper:SolderJumper-2_P1.3mm_Open_RoundedPad1.0x1.5mm" H 6300 6400 50  0001 C CNN
-F 3 "~" H 6300 6400 50  0001 C CNN
-	1    6300 6400
-	0    1    1    0
-$EndComp
-$Comp
-L Device:R R53
-U 1 1 5D60D82D
-P 6300 6850
-F 0 "R53" V 6093 6850 50  0000 C CNN
-F 1 "10K" V 6184 6850 50  0000 C CNN
-F 2 "Resistor_SMD:R_0201_0603Metric" V 6230 6850 50  0001 C CNN
-F 3 "~" H 6300 6850 50  0001 C CNN
-	1    6300 6850
-	-1   0    0    1
-$EndComp
 $Comp
 L power:GND #PWR0241
@@
 Text Notes 7700 7000 0    50   ~ 0
 Normal boot mode: boot from fuses\n-----------------------------------\n\nGPIO boot override pins are ignored. The boot ROM code uses the boot \neFUSE settings only. This mode also supports a secure boot using HAB.\n\nUnprogrammed device boot flow (BT_FUSE_SEL = 0)\n-----------------------------------\n\n- Boot ROM detect SD/MMC card on USDHC2 port. If a card is inserted, \nROM will try to boot from it. This is the so-called Manufacture SD/MMC\nboot. This feature can be disabled by blowing fuse “Disable SD/MMC \nManufacture Mode”.\n- Subsequently jumps to the Serial Downloader\n\nProgrammed device boot flow (BT_FUSE_SEL = 1)\n-----------------------------------\n\n- Boot from eMMC (USDHC1)\n- If not programmed fall back to SD (USDHC2)\n- Fall back to Serial Downloader
+Text Label 6000 6600 0    50   ~ 0
+BTN0
 $EndSCHEMATC

Commit message: Add esd protection for usb
Connections:
- net VDD_1V8: no longer R43.1, R44.1, R47.1, R48.1
- net VDD_3V3: now also R43.1, R44.1, R47.1, R48.1
Other:
- note added: "EN - output, 3.3v push-pull\nOC - input, internal pull-up"
- note added: "WDOG - input, internal pull-up\nnINT - input, internal pull-up\nVSEL - output, 1.8v push-pull"
Changed lines of the file:
@@
 Text Label 1700 3350 0    50   ~ 0
 I2C2_SDA
-Text Label 15650 7100 0    50   ~ 0
+Text Label 15650 7350 0    50   ~ 0
 I2C3_SCL
-Text Label 15650 7200 0    50   ~ 0
+Text Label 15650 7450 0    50   ~ 0
 I2C3_SDA
 Wire Wire Line
-	15650 7100 15500 7100
-Wire Wire Line
-	15650 7200 15550 7200
-Wire Wire Line
-	15500 7100 15500 7350
-Wire Wire Line
 	15500 7350 15400 7350
-Connection ~ 15500 7100
-Wire Wire Line
-	15500 7100 15400 7100
 Wire Wire Line
 	15500 7350 15500 7600
 Wire Wire Line
 	15500 7600 15400 7600
-Connection ~ 15500 7350
-Wire Wire Line
-	15550 7200 15550 7450
 Wire Wire Line
 	15550 7450 15400 7450
-Connection ~ 15550 7200
-Wire Wire Line
-	15550 7200 15400 7200
 Wire Wire Line
 	15550 7450 15550 7700
 Wire Wire Line
 	15550 7700 15400 7700
-Connection ~ 15550 7450
 Text Label 13100 7600 2    50   ~ 0
 DP_SUSP
@@
 	10300 8100 10300 7950
 Wire Wire Line
-	10400 7950 10600 7950
-Connection ~ 10400 7950
-Wire Wire Line
 	10400 8100 10400 7950
 Wire Wire Line
 	10600 7950 10700 7950
-Connection ~ 10600 7950
 Wire Wire Line
 	10600 8400 10600 7950
@@
 Text Label 6000 6600 0    50   ~ 0
 BTN0
+Text Notes 2450 4200 0    35   ~ 0
+EN - output, 3.3v push-pull\nOC - input, internal pull-up
+Text Notes 6050 2950 0    35   ~ 0
+WDOG - input, internal pull-up\nnINT - input, internal pull-up\nVSEL - output, 1.8v push-pull
+Wire Wire Line
+	15400 7100 15650 7100
+Wire Wire Line
+	15400 7200 15650 7200
+Wire Wire Line
+	15650 7350 15500 7350
+Connection ~ 15500 7350
+Wire Wire Line
+	15550 7450 15650 7450
+Connection ~ 15550 7450
+$Comp
+L mxenc:VDD_3V3 #PWR0142
+U 1 1 5DC891CB
+P 10600 7850
+F 0 "#PWR0142" H 10600 7700 50  0001 C CNN
+F 1 "VDD_3V3" H 10615 8023 50  0000 C CNN
+F 2 "" H 10600 7850 50  0001 C CNN
+F 3 "" H 10600 7850 50  0001 C CNN
+	1    10600 7850
+	1    0    0    -1
+$EndComp
+Wire Wire Line
+	10600 7850 10600 7950
+Connection ~ 10600 7950
+Text Label 15650 7100 0    50   ~ 0
+I2C2_SCL
+Text Label 15650 7200 0    50   ~ 0
+I2C2_SDA
 $EndSCHEMATC

Commit message: Re-add gg logo
Parts:
- added L8: GG_LOGO, mxenc:gg-4x4, symbol mxenc:GG_LOGO
Changed lines of the file:
@@
 Text Label 15650 7200 0    50   ~ 0
 I2C2_SDA
+$Comp
+L mxenc:GG_LOGO L8
+U 1 1 5DF62B5A
+P 11750 10350
+F 0 "L8" H 11800 10395 50  0000 L CNN
+F 1 "GG_LOGO" H 11800 10304 50  0000 L CNN
+F 2 "mxenc:gg-4x4" H 11750 10350 50  0001 C CNN
+F 3 "" H 11750 10350 50  0001 C CNN
+	1    11750 10350
+	1    0    0    -1
+$EndComp
 $EndSCHEMATC

Commit message: Complete entry of bom
Parts:
- C166, C167: Mfgr (none) -> TDK; Part (none) -> CGA1A2C0G1E120J030BA; Vendorpart (none) -> 445-9070-1-ND
- D1: Mfgr (none) -> Broadcom; Part (none) -> ASMB-KTF0-0A306
- J4, J6: Mfgr (none) -> JST; Part (none) -> SM06B-GHS-TB(LF)(SN); Vendorpart (none) -> 455-1568-1-ND
- J8: value Conn_01x06 -> Conn_01x06 DNP
- R35: Mfgr (none) -> Yageo; Part (none) -> RC0201FR-07510KL; Vendorpart (none) -> YAG2713CT-ND
- R41, R42, R43, R44, R45, R46, R47, R48: Mfgr (none) -> Yageo; Part (none) -> RC0201JR-074K7L; Vendorpart (none) -> 311-4.7KNCT-ND
- R52, R54, R58: Mfgr (none) -> Panasonic; Part (none) -> ERJ-1GNJ103C; Vendorpart (none) -> P123222CT-ND
- R55: Mfgr (none) -> Yageo; Part (none) -> RC0201JR-0768RL; Vendorpart (none) -> YAG2364CT-ND
- R56, R57: Mfgr (none) -> Yageo; Part (none) -> RC0201JR-0722RL; Vendorpart (none) -> 311-22NCT-ND
- R59: Mfgr (none) -> Yageo; Part (none) -> RC0201JR-07100KL; Vendorpart (none) -> 311-100KNCT-ND
- SW1, SW2: Mfgr (none) -> C&K; Part (none) -> PTS810 SJK 250 SMTR LFS; Vendorpart (none) -> CKN10503CT-ND
- U1: value MIMX8MM6DVTLZAA -> IMX8MM; Mfgr (none) -> NXP; Part (none) -> MIMX8MM6CVTKZAA; Vendorpart (none) -> 568-15276-ND
- U10: Mfgr (none) -> Microchip; Part (none) -> 24LC16B-I/MC; Vendorpart (none) -> 24LC16B-I/MC-ND
- Y2: Mfgr (none) -> Murata; Part (none) -> XRCGB24M000F0L00R0; Vendorpart (none) -> 490-5575-1-ND
Changed lines of the file:
@@
 F 2 "Button_Switch_SMD:SW_SPST_PTS810" H 8750 1400 50  0001 C CNN
 F 3 "~" H 8750 1400 50  0001 C CNN
+F 4 "CKN10503CT-ND" H 8750 1200 50  0000 C CNN "Vendorpart"
+F 5 "C&K" H 8750 1200 50  0001 C CNN "Mfgr"
+F 6 "PTS810 SJK 250 SMTR LFS" H 8750 1200 50  0001 C CNN "Part"
 	1    8750 1200
 	1    0    0    -1
@@
 F 2 "Button_Switch_SMD:SW_SPST_PTS810" H 8750 2000 50  0001 C CNN
 F 3 "~" H 8750 2000 50  0001 C CNN
+F 4 "CKN10503CT-ND" H 8750 1800 50  0000 C CNN "Vendorpart"
+F 5 "C&K" H 8750 1800 50  0001 C CNN "Mfgr"
+F 6 "PTS810 SJK 250 SMTR LFS" H 8750 1800 50  0001 C CNN "Part"
 	1    8750 1800
 	1    0    0    -1
@@
 F 2 "Connector_JST:JST_GH_SM06B-GHS-TB_1x06-1MP_P1.25mm_Horizontal" H 2250 1400 50  0001 C CNN
 F 3 "~" H 2250 1400 50  0001 C CNN
+F 4 "455-1568-1-ND" H 2250 1400 50  0000 C CNN "Vendorpart"
+F 5 "JST" H 2250 1400 50  0001 C CNN "Mfgr"
+F 6 "SM06B-GHS-TB(LF)(SN)" H 2250 1400 50  0001 C CNN "Part"
 	1    2250 1400
 	1    0    0    -1
@@
 F 2 "Package_DFN_QFN:DFN-8-1EP_3x2mm_P0.5mm_EP1.36x1.46mm" H 1100 3450 50  0001 C CNN
 F 3 "http://ww1.microchip.com/downloads/en/DeviceDoc/21703d.pdf" H 1100 3450 50  0001 C CNN
+F 4 "Microchip" H 1100 3450 50  0001 C CNN "Mfgr"
+F 5 "24LC16B-I/MC" H 1100 3450 50  0001 C CNN "Part"
+F 6 "24LC16B-I/MC-ND" H 1100 3450 50  0001 C CNN "Vendorpart"
 	1    1100 3450
 	1    0    0    -1
@@
 P 4550 5250
 F 0 "U1" H 4575 8115 50  0000 C CNN
-F 1 "MIMX8MM6DVTLZAA" H 4575 8024 50  0000 C CNN
+F 1 "IMX8MM" H 4575 8024 50  0000 C CNN
 F 2 "mxenc:BGA-729_27x27_14.0x14.0mm" H 4800 8000 50  0001 C CNN
 F 3 "" H 3800 8000 50  0001 C CNN
+F 4 "568-15276-ND" H 4550 5250 50  0000 C CNN "Vendorpart"
+F 5 "NXP" H 4550 5250 50  0001 C CNN "Mfgr"
+F 6 "MIMX8MM6CVTKZAA" H 4550 5250 50  0001 C CNN "Part"
 	11   4550 5250
 	1    0    0    -1
@@
 F 2 "Resistor_SMD:R_0201_0603Metric" V 6080 4050 50  0001 C CNN
 F 3 "~" H 6150 4050 50  0001 C CNN
+F 4 "P123222CT-ND" H 6150 4050 50  0000 C CNN "Vendorpart"
+F 5 "Panasonic" H 6150 4050 50  0001 C CNN "Mfgr"
+F 6 "ERJ-1GNJ103C" H 6150 4050 50  0001 C CNN "Part"
 	1    6150 4050
 	-1   0    0    1
@@
 F 2 "Resistor_SMD:R_0201_0603Metric" V 6380 4050 50  0001 C CNN
 F 3 "~" H 6450 4050 50  0001 C CNN
+F 4 "Panasonic" H 6450 4050 50  0001 C CNN "Mfgr"
+F 5 "ERJ-1GNJ103C" H 6450 4050 50  0001 C CNN "Part"
+F 6 "P123222CT-ND" H 6450 4050 50  0001 C CNN "Vendorpart"
 	1    6450 4050
 	-1   0    0    1
@@
 F 3 "~" H 7450 1450 50  0001 C CNN
 F 4 "516-3906-1-ND" H 7450 1905 50  0000 C CNN "Vendorpart"
+F 5 "Broadcom" H 7450 1500 50  0001 C CNN "Mfgr"
+F 6 "ASMB-KTF0-0A306" H 7450 1500 50  0001 C CNN "Part"
 	1    7450 1500
 	1    0    0    -1
@@
 P 9050 1850
 F 0 "U1" H 9050 2650 50  0000 C CNN
-F 1 "MIMX8MM6DVTLZAA" H 9000 2750 50  0000 C CNN
+F 1 "IMX8MM" H 9000 2750 50  0000 C CNN
 F 2 "mxenc:BGA-729_27x27_14.0x14.0mm" H 9300 4600 50  0001 C CNN
 F 3 "" H 8300 4600 50  0001 C CNN
+F 4 "NXP" H 9050 1850 50  0001 C CNN "Mfgr"
+F 5 "MIMX8MM6CVTKZAA" H 9050 1850 50  0001 C CNN "Part"
+F 6 "568-15276-ND" H 9050 1850 50  0001 C CNN "Vendorpart"
 	7    9050 1850
 	-1   0    0    1
@@
 F 2 "Resistor_SMD:R_0201_0603Metric" V 6880 1300 50  0001 C CNN
 F 3 "~" H 6950 1300 50  0001 C CNN
+F 4 "Yageo" H 6950 1300 50  0001 C CNN "Mfgr"
+F 5 "RC0201JR-0768RL" H 6950 1300 50  0001 C CNN "Part"
+F 6 "YAG2364CT-ND" H 6950 1300 50  0001 C CNN "Vendorpart"
 	1    6950 1300
 	0    -1   -1   0
@@
 F 2 "Resistor_SMD:R_0201_0603Metric" V 6880 1500 50  0001 C CNN
 F 3 "~" H 6950 1500 50  0001 C CNN
+F 4 "Yageo" H 6950 1500 50  0001 C CNN "Mfgr"
+F 5 "RC0201JR-0722RL" H 6950 1500 50  0001 C CNN "Part"
+F 6 "311-22NCT-ND" H 6950 1500 50  0001 C CNN "Vendorpart"
 	1    6950 1500
 	0    -1   -1   0
@@
 F 2 "Resistor_SMD:R_0201_0603Metric" V 6880 1700 50  0001 C CNN
 F 3 "~" H 6950 1700 50  0001 C CNN
+F 4 "Yageo" H 6950 1700 50  0001 C CNN "Mfgr"
+F 5 "RC0201JR-0722RL" H 6950 1700 50  0001 C CNN "Part"
+F 6 "311-22NCT-ND" H 6950 1700 50  0001 C CNN "Vendorpart"
 	1    6950 1700
 	0    -1   -1   0
@@
 F 2 "Connector_JST:JST_GH_SM06B-GHS-TB_1x06-1MP_P1.25mm_Horizontal" H 3700 1400 50  0001 C CNN
 F 3 "~" H 3700 1400 50  0001 C CNN
+F 4 "455-1568-1-ND" H 3700 1400 50  0000 C CNN "Vendorpart"
+F 5 "JST" H 3700 1400 50  0001 C CNN "Mfgr"
+F 6 "SM06B-GHS-TB(LF)(SN)" H 3700 1400 50  0001 C CNN "Part"
 	1    3700 1400
 	1    0    0    -1
@@
 P 5400 1400
 F 0 "J8" H 5480 1392 50  0000 L CNN
-F 1 "Conn_01x06" H 5480 1301 50  0000 L CNN
+F 1 "Conn_01x06 DNP" H 5480 1301 50  0000 L CNN
 F 2 "Connector_PinHeader_2.54mm:PinHeader_1x06_P2.54mm_Horizontal" H 5400 1400 50  0001 C CNN
 F 3 "~" H 5400 1400 50  0001 C CNN
@@
 P 3850 9350
 F 0 "U1" H 3850 12215 50  0000 C CNN
-F 1 "MIMX8MM6DVTLZAA" H 3850 12124 50  0000 C CNN
+F 1 "IMX8MM" H 3850 12124 50  0000 C CNN
 F 2 "mxenc:BGA-729_27x27_14.0x14.0mm" H 4100 12100 50  0001 C CNN
 F 3 "" H 3100 12100 50  0001 C CNN
+F 4 "NXP" H 3850 9350 50  0001 C CNN "Mfgr"
+F 5 "MIMX8MM6CVTKZAA" H 3850 9350 50  0001 C CNN "Part"
+F 6 "568-15276-ND" H 3850 9350 50  0001 C CNN "Vendorpart"
 	12   3850 9350
 	1    0    0    -1
@@
 F 2 "Resistor_SMD:R_0201_0603Metric" V 5430 8000 50  0001 C CNN
 F 3 "~" H 5500 8000 50  0001 C CNN
+F 4 "Yageo" H 5500 8000 50  0001 C CNN "Mfgr"
+F 5 "RC0201JR-07100KL" H 5500 8000 50  0001 C CNN "Part"
+F 6 "311-100KNCT-ND" H 5500 8000 50  0001 C CNN "Vendorpart"
 	1    5500 8000
 	0    -1   -1   0
@@
 F 2 "Resistor_SMD:R_0201_0603Metric" V 2180 6650 50  0001 C CNN
 F 3 "~" H 2250 6650 50  0001 C CNN
+F 4 "Panasonic" H 2250 6650 50  0001 C CNN "Mfgr"
+F 5 "ERJ-1GNJ103C" H 2250 6650 50  0001 C CNN "Part"
+F 6 "P123222CT-ND" H 2250 6650 50  0001 C CNN "Vendorpart"
 	1    2250 6650
 	-1   0    0    1
@@
 F 2 "Resistor_SMD:R_0201_0603Metric" V 1780 8300 50  0001 C CNN
 F 3 "~" H 1850 8300 50  0001 C CNN
+F 4 "Yageo" H 1850 8300 50  0001 C CNN "Mfgr"
+F 5 "RC0201FR-07510KL" H 1850 8300 50  0001 C CNN "Part"
+F 6 "YAG2713CT-ND" H 1850 8300 50  0001 C CNN "Vendorpart"
 	1    1850 8300
 	0    1    1    0
@@
 F 2 "Capacitor_SMD:C_0201_0603Metric" H 2288 8850 50  0001 C CNN
 F 3 "~" H 2250 9000 50  0001 C CNN
+F 4 "TDK" H 2250 9000 50  0001 C CNN "Mfgr"
+F 5 "CGA1A2C0G1E120J030BA" H 2250 9000 50  0001 C CNN "Part"
+F 6 "445-9070-1-ND" H 2250 9000 50  0001 C CNN "Vendorpart"
 	1    2250 9000
 	1    0    0    -1
@@
 F 2 "Capacitor_SMD:C_0201_0603Metric" H 1488 8850 50  0001 C CNN
 F 3 "~" H 1450 9000 50  0001 C CNN
+F 4 "TDK" H 1450 9000 50  0001 C CNN "Mfgr"
+F 5 "CGA1A2C0G1E120J030BA" H 1450 9000 50  0001 C CNN "Part"
+F 6 "445-9070-1-ND" H 1450 9000 50  0001 C CNN "Vendorpart"
 	1    1450 9000
 	1    0    0    -1
@@
 F 2 "mxenc:XRCGB" H 1850 8700 50  0001 C CNN
 F 3 "~" H 1850 8700 50  0001 C CNN
+F 4 "Murata" H 1850 8700 50  0001 C CNN "Mfgr"
+F 5 "XRCGB24M000F0L00R0" H 1850 8700 50  0001 C CNN "Part"
+F 6 "490-5575-1-ND" H 1850 8700 50  0001 C CNN "Vendorpart"
 	1    1850 8700
 	1    0    0    -1
@@
 F 2 "Resistor_SMD:R_0201_0603Metric" V 10930 8250 50  0001 C CNN
 F 3 "~" H 11000 8250 50  0001 C CNN
+F 4 "Yageo" H 11000 8250 50  0001 C CNN "Mfgr"
+F 5 "RC0201JR-074K7L" H 11000 8250 50  0001 C CNN "Part"
+F 6 "311-4.7KNCT-ND" H 11000 8250 50  0001 C CNN "Vendorpart"
 	1    11000 8250
 	1    0    0    -1
@@
 F 2 "Resistor_SMD:R_0201_0603Metric" V 10830 8250 50  0001 C CNN
 F 3 "~" H 10900 8250 50  0001 C CNN
+F 4 "Yageo" H 10900 8250 50  0001 C CNN "Mfgr"
+F 5 "RC0201JR-074K7L" H 10900 8250 50  0001 C CNN "Part"
+F 6 "311-4.7KNCT-ND" H 10900 8250 50  0001 C CNN "Vendorpart"
 	1    10900 8250
 	-1   0    0    -1
@@
 F 2 "Resistor_SMD:R_0201_0603Metric" V 10330 8250 50  0001 C CNN
 F 3 "~" H 10400 8250 50  0001 C CNN
+F 4 "Yageo" H 10400 8250 50  0001 C CNN "Mfgr"
+F 5 "RC0201JR-074K7L" H 10400 8250 50  0001 C CNN "Part"
+F 6 "311-4.7KNCT-ND" H 10400 8250 50  0001 C CNN "Vendorpart"
 	1    10400 8250
 	1    0    0    -1
@@
 F 2 "Resistor_SMD:R_0201_0603Metric" V 10230 8250 50  0001 C CNN
 F 3 "~" H 10300 8250 50  0001 C CNN
+F 4 "Yageo" H 10300 8250 50  0001 C CNN "Mfgr"
+F 5 "RC0201JR-074K7L" H 10300 8250 50  0001 C CNN "Part"
+F 6 "311-4.7KNCT-ND" H 10300 8250 50  0001 C CNN "Vendorpart"
 	1    10300 8250
 	-1   0    0    -1
@@
 F 2 "Resistor_SMD:R_0201_0603Metric" V 10630 8550 50  0001 C CNN
 F 3 "~" H 10700 8550 50  0001 C CNN
+F 4 "Yageo" H 10700 8550 50  0001 C CNN "Mfgr"
+F 5 "RC0201JR-074K7L" H 10700 8550 50  0001 C CNN "Part"
+F 6 "311-4.7KNCT-ND" H 10700 8550 50  0001 C CNN "Vendorpart"
 	1    10700 8550
 	1    0    0    -1
@@
 F 2 "Resistor_SMD:R_0201_0603Metric" V 10530 8550 50  0001 C CNN
 F 3 "~" H 10600 8550 50  0001 C CNN
+F 4 "Yageo" H 10600 8550 50  0001 C CNN "Mfgr"
+F 5 "RC0201JR-074K7L" H 10600 8550 50  0001 C CNN "Part"
+F 6 "311-4.7KNCT-ND" H 10600 8550 50  0001 C CNN "Vendorpart"
 	1    10600 8550
 	-1   0    0    -1
@@
 F 2 "Resistor_SMD:R_0201_0603Metric" V 10030 8550 50  0001 C CNN
 F 3 "~" H 10100 8550 50  0001 C CNN
+F 4 "Yageo" H 10100 8550 50  0001 C CNN "Mfgr"
+F 5 "RC0201JR-074K7L" H 10100 8550 50  0001 C CNN "Part"
+F 6 "311-4.7KNCT-ND" H 10100 8550 50  0001 C CNN "Vendorpart"
 	1    10100 8550
 	1    0    0    -1
@@
 F 2 "Resistor_SMD:R_0201_0603Metric" V 9930 8550 50  0001 C CNN
 F 3 "~" H 10000 8550 50  0001 C CNN
+F 4 "Yageo" H 10000 8550 50  0001 C CNN "Mfgr"
+F 5 "RC0201JR-074K7L" H 10000 8550 50  0001 C CNN "Part"
+F 6 "311-4.7KNCT-ND" H 10000 8550 50  0001 C CNN "Vendorpart"
 	1    10000 8550
 	-1   0    0    -1
@@
 P 8550 11400
 F 0 "U1" H 8550 14265 50  0000 C CNN
-F 1 "MIMX8MM6DVTLZAA" H 8550 14174 50  0000 C CNN
+F 1 "IMX8MM" H 8550 14174 50  0000 C CNN
 F 2 "mxenc:BGA-729_27x27_14.0x14.0mm" H 8800 14150 50  0001 C CNN
 F 3 "" H 7800 14150 50  0001 C CNN
+F 4 "NXP" H 8550 11400 50  0001 C CNN "Mfgr"
+F 5 "MIMX8MM6CVTKZAA" H 8550 11400 50  0001 C CNN "Part"
+F 6 "568-15276-ND" H 8550 11400 50  0001 C CNN "Vendorpart"
 	6    8550 11400
 	1    0    0    -1

Commit message: wip
Parts:
- added J9: Conn_02x35_Odd_Even, mxenc:DF40HC(3.0)-70DS, symbol Connector_Generic:Conn_02x35_Odd_Even
Changed lines of the file:
@@
+	1    0    0    -1
+$EndComp
+$Comp
+L Connector_Generic:Conn_02x35_Odd_Even J9
+U 1 1 5E041DEE
+P 11550 6000
+F 0 "J9" H 11600 7917 50  0000 C CNN
+F 1 "Conn_02x35_Odd_Even" H 11600 7826 50  0000 C CNN
+F 2 "mxenc:DF40HC(3.0)-70DS" H 11550 6000 50  0001 C CNN
+F 3 "~" H 11550 6000 50  0001 C CNN
+	1    11550 6000
 	1    0    0    -1
 $EndComp

Commit message: wip more new layout
Parts:
- removed J9: Conn_02x35_Odd_Even, mxenc:DF40HC(3.0)-70DS, symbol Connector_Generic:Conn_02x35_Odd_Even
Changed lines of the file:
@@
 $Descr USLedger 17000 11000
 encoding utf-8
-Sheet 1 9
+Sheet 1 10
 Title ""
 Date ""
@@
 F1 "USB.sch" 50
 F2 "LD1_~INT" I L 13350 6850 50
-F3 "USB2_VBUS_IN" O L 13350 6950 50
+F3 "USB1_VBUS_IN" O L 13350 6950 50
 F4 "USB1_VBUS_OC" O L 13350 7300 50
 F5 "USB1_VBUS_EN" I L 13350 7400 50
@@
 F10 "USB2_SCL" I R 15400 7350 50
 F11 "USB2_SDA" B R 15400 7450 50
-F12 "USB2_PWR_SDA" B R 15400 7700 50
-F13 "USB2_PWR_SCL" I R 15400 7600 50
+F12 "USB1_PWR_SDA" B R 15400 7700 50
+F13 "USB1_PWR_SCL" I R 15400 7600 50
 F14 "DP_SUSP" I L 13350 7600 50
 $EndSheet
@@
 Text Notes 4200 6300 0    50   ~ 0
 BOOT_MODE[1:0] == 00 :: Boot from fuses\nBOOT_MODE[1:0] == 01 :: Serial downloader
-Text Notes 7700 7000 0    50   ~ 0
+Text Notes 7200 7050 0    50   ~ 0
 Normal boot mode: boot from fuses\n-----------------------------------\n\nGPIO boot override pins are ignored. The boot ROM code uses the boot \neFUSE settings only. This mode also supports a secure boot using HAB.\n\nUnprogrammed device boot flow (BT_FUSE_SEL = 0)\n-----------------------------------\n\n- Boot ROM detect SD/MMC card on USDHC2 port. If a card is inserted, \nROM will try to boot from it. This is the so-called Manufacture SD/MMC\nboot. This feature can be disabled by blowing fuse “Disable SD/MMC \nManufacture Mode”.\n- Subsequently jumps to the Serial Downloader\n\nProgrammed device boot flow (BT_FUSE_SEL = 1)\n-----------------------------------\n\n- Boot from eMMC (USDHC1)\n- If not programmed fall back to SD (USDHC2)\n- Fall back to Serial Downloader
 Text Label 6000 6600 0    50   ~ 0
@@
 	1    0    0    -1
 $EndComp
-$Comp
-L Connector_Generic:Conn_02x35_Odd_Even J9
-U 1 1 5E041DEE
-P 11550 6000
-F 0 "J9" H 11600 7917 50  0000 C CNN
-F 1 "Conn_02x35_Odd_Even" H 11600 7826 50  0000 C CNN
-F 2 "mxenc:DF40HC(3.0)-70DS" H 11550 6000 50  0001 C CNN
-F 3 "~" H 11550 6000 50  0001 C CNN
-	1    11550 6000
-	1    0    0    -1
-$EndComp
+$Sheet
+S 11000 5550 1450 850
+U 5E34BAA5
+F0 "Expansion" 50
+F1 "expansion.sch" 50
+$EndSheet
 $EndSCHEMATC
