File: hardware_sbc/CPU-power.sch (KiCad schematic (older format))
At the start: 57 parts, among them U1 IMX8MM

Commit message: BOM and misc fixes for production of 0.9 boards
Parts:
- C29, C41, C47, C57, C58, C65, C72, C73: Mfgrpart (none) -> GRM155C80J106ME11D; Part GRM155C80J106ME11D -> (none)
- C30, C31, C32, C34, C35, C37, C38, C39, C40, C53, C54, C55, C56, C66, C67, C68, C69, C71, C80, C81: Mfgrpart (none) -> GRM033C80J224KE90D; Part GRM033C80J224KE90D -> (none)
- C33, C42, C43, C44, C45, C46, C48, C49, C50, C51, C52, C59, C60, C61, C62, C63, C64, C74, C75, C76, C77, C78, C79, C84: Mfgrpart (none) -> GRM033C80G105ME05D; Part GRM033C80G105ME05D -> (none)
- C36, C70: Mfgrpart (none) -> GRM155C80J475MEAAD; Part GRM155C80J475MEAAD -> (none)
- C82: Mfgrpart (none) -> GRM033D80E225ME47D; Part GRM033D80E225ME47D -> (none)
- C83: Mfgrpart (none) -> GRM033R70J222KA01D; Part GRM033R70J222KA01D -> (none)
- U1: Mfgrpart (none) -> MIMX8MM6CVTKZAA; Part MIMX8MM6CVTKZAA -> (none)
