File: hardware_sbc/DRAM.sch (KiCad schematic (older format))
At the start: 38 parts, among them U1 IMX8MM, U3 MT53E256M32D2DS-053 WT:B

Commit message: Clean up bom and add config for KiBoM
Parts:
- U3: Part MT53E256M32D2DS-053 WT:B -> MT53D512M32D2DS-053 WT:D; Vendor Mouser -> Arrow; Vendorpart 340-359530 -> MT53D512M32D2DS-053 WT:D
Changed lines of the file:
@@
 F 3 "" H 10700 4650 50  0001 L BNN
 F 4 "Micron" H 10700 4650 50  0001 C CNN "Mfgr"
-F 5 "MT53E256M32D2DS-053 WT:B" H 10700 4650 50  0001 C CNN "Part"
-F 6 "340-359530" H 10700 4650 50  0001 C CNN "Vendorpart"
-F 7 "Mouser" H 10700 4650 50  0001 C CNN "Vendor"
+F 5 "MT53D512M32D2DS-053 WT:D" H 10700 4650 50  0001 C CNN "Part"
+F 6 "MT53D512M32D2DS-053 WT:D" H 10700 4650 50  0001 C CNN "Vendorpart"
+F 7 "Arrow" H 10700 4650 50  0001 C CNN "Vendor"
 	1    10700 4650
 	1    0    0    -1

Commit message: BOM and misc fixes for production of 0.9 boards
Parts:
- C10, C15, C16, C17, C18, C19, C24, C25, C26, C27, C28, C7, C8, C9: Mfgrpart (none) -> GRM155C8YA224ME01D; Part GRM155C8YA224ME01D -> (none)
- C11, C12, C13, C14, C20, C21, C22, C23, C3, C4, C5, C6: Mfgrpart (none) -> GRM155C80J106ME11D; Part GRM155C80J106ME11D -> (none)
- R21, R22, R23, R27, R28: Mfgrpart (none) -> ERJ-2GEJ103X; Part ERJ-2GEJ103X -> (none)
- R24, R25, R26: Mfgrpart (none) -> RC0402FR-07240RP; Part RC0402FR-07240RP -> (none)
- R29, R30: Mfgrpart (none) -> RC0402FR-07150RL; Part RC0402FR-07150RL -> (none)
- U1: Mfgrpart (none) -> MIMX8MM6CVTKZAA; Part MIMX8MM6CVTKZAA -> (none)
- U3: Mfgrpart (none) -> MT53D512M32D2DS-053 WT:D; Part MT53D512M32D2DS-053 WT:D -> (none)
