File: hardware_sbc/PMIC.sch (KiCad schematic (older format))
At the start: 60 parts, among them U4 BD71847MWV, Y2 Crystal

Commit message: BOM and misc fixes for production of 0.9 boards
Parts:
- C100, C104, C117, C118, C87, C93, C97: Mfgrpart (none) -> GRM155C81A105KA12D; Part GRM155C81A105KA12D -> (none)
- C101, C102, C106, C107, C110, C111, C115, C116, C91, C92, C95, C96: Mfgrpart (none) -> GRM188C80G226MEA0D; Part GRM188C80G226MEA0D -> (none)
- C103, C105, C109, C112, C85, C86, C94, C98: Mfgrpart (none) -> CL10X106MO8NRNC; Part CL10X106MO8NRNC -> (none)
- C108, C114, C99: Mfgrpart (none) -> GRM155C80J475MEAAD; Part GRM155C80J475MEAAD -> (none)
- C113: Mfgrpart (none) -> CL10B105MO8NNWC; Part CL10B105MO8NNWC -> (none)
- C119, C120: Mfgrpart (none) -> GRM0335C1H180JA01D; Part GRM0335C1H180JA01D -> (none)
- C88, C89, C90: Mfgrpart (none) -> GRM155C80J225ME95D; Part GRM155C80J225ME95D -> (none)
- L2, L3, L4, L6, L7: Mfgrpart (none) -> CIGT201610EHR47MNE; Part CIGT201610EHR47MNE -> (none)
- L5: Mfgrpart (none) -> CIGT201610EH1R0MNE; Part CIGT201610EH1R0MNE -> (none)
- R31, R32: Mfgrpart (none) -> RC0402JR-07100KL; Part RC0402JR-07100KL -> (none)
- U4: Mfgrpart (none) -> BD71847AMWV-E2; Part BD71847AMWV-E2 -> (none)
- Y2: Mfgrpart (none) -> ABS07-32.768KHZ-T; Part ABS07-32.768KHZ-T -> (none)
