File: hardware_sbc/PMIC.sch (KiCad schematic (older format))
At the start: 60 parts, among them U4 BD71847MWV, Y2 Crystal

Commit message: Change common 22uF part from 4V to 6.3V
Most placements don't require 5V, but a few do. The 4V part is no
longer stocking as well, and price is similar, so change all to
6.3V version.
Parts:
- C101, C102, C106, C107, C110, C111, C115, C116, C91, C92, C95, C96: Mfgrpart GRM188C80G226MEA0D -> GRM188C80J226ME15D; Vendorpart 490-7196-1-ND -> 490-10471-1-ND
Changed lines of the file:
@@
 F 4 "Murata" H 6000 1850 50  0001 C CNN "Mfgr"
 F 5 "" H 6000 1850 50  0001 C CNN "Part"
-F 6 "490-7196-1-ND" H 6000 1850 50  0001 C CNN "Vendorpart"
-F 7 "GRM188C80G226MEA0D" H 6000 1850 50  0001 C CNN "Mfgrpart"
+F 6 "490-10471-1-ND" H 6000 1850 50  0001 C CNN "Vendorpart"
+F 7 "GRM188C80J226ME15D" H 6000 1850 50  0001 C CNN "Mfgrpart"
 	1    6000 1850
 	-1   0    0    1
@@
 F 4 "Murata" H 6300 1850 50  0001 C CNN "Mfgr"
 F 5 "" H 6300 1850 50  0001 C CNN "Part"
-F 6 "490-7196-1-ND" H 6300 1850 50  0001 C CNN "Vendorpart"
-F 7 "GRM188C80G226MEA0D" H 6300 1850 50  0001 C CNN "Mfgrpart"
+F 6 "490-10471-1-ND" H 6300 1850 50  0001 C CNN "Vendorpart"
+F 7 "GRM188C80J226ME15D" H 6300 1850 50  0001 C CNN "Mfgrpart"
 	1    6300 1850
 	-1   0    0    1
@@
 F 4 "Murata" H 6000 2300 50  0001 C CNN "Mfgr"
 F 5 "" H 6000 2300 50  0001 C CNN "Part"
-F 6 "490-7196-1-ND" H 6000 2300 50  0001 C CNN "Vendorpart"
-F 7 "GRM188C80G226MEA0D" H 6000 2300 50  0001 C CNN "Mfgrpart"
+F 6 "490-10471-1-ND" H 6000 2300 50  0001 C CNN "Vendorpart"
+F 7 "GRM188C80J226ME15D" H 6000 2300 50  0001 C CNN "Mfgrpart"
 	1    6000 2300
 	-1   0    0    1
@@
 F 4 "Murata" H 6300 2300 50  0001 C CNN "Mfgr"
 F 5 "" H 6300 2300 50  0001 C CNN "Part"
-F 6 "490-7196-1-ND" H 6300 2300 50  0001 C CNN "Vendorpart"
-F 7 "GRM188C80G226MEA0D" H 6300 2300 50  0001 C CNN "Mfgrpart"
+F 6 "490-10471-1-ND" H 6300 2300 50  0001 C CNN "Vendorpart"
+F 7 "GRM188C80J226ME15D" H 6300 2300 50  0001 C CNN "Mfgrpart"
 	1    6300 2300
 	-1   0    0    1
@@
 F 4 "Murata" H 6000 2750 50  0001 C CNN "Mfgr"
 F 5 "" H 6000 2750 50  0001 C CNN "Part"
-F 6 "490-7196-1-ND" H 6000 2750 50  0001 C CNN "Vendorpart"
-F 7 "GRM188C80G226MEA0D" H 6000 2750 50  0001 C CNN "Mfgrpart"
+F 6 "490-10471-1-ND" H 6000 2750 50  0001 C CNN "Vendorpart"
+F 7 "GRM188C80J226ME15D" H 6000 2750 50  0001 C CNN "Mfgrpart"
 	1    6000 2750
 	-1   0    0    1
@@
 F 4 "Murata" H 6300 2750 50  0001 C CNN "Mfgr"
 F 5 "" H 6300 2750 50  0001 C CNN "Part"
-F 6 "490-7196-1-ND" H 6300 2750 50  0001 C CNN "Vendorpart"
-F 7 "GRM188C80G226MEA0D" H 6300 2750 50  0001 C CNN "Mfgrpart"
+F 6 "490-10471-1-ND" H 6300 2750 50  0001 C CNN "Vendorpart"
+F 7 "GRM188C80J226ME15D" H 6300 2750 50  0001 C CNN "Mfgrpart"
 	1    6300 2750
 	-1   0    0    1
@@
 F 4 "Murata" H 6000 3200 50  0001 C CNN "Mfgr"
 F 5 "" H 6000 3200 50  0001 C CNN "Part"
-F 6 "490-7196-1-ND" H 6000 3200 50  0001 C CNN "Vendorpart"
-F 7 "GRM188C80G226MEA0D" H 6000 3200 50  0001 C CNN "Mfgrpart"
+F 6 "490-10471-1-ND" H 6000 3200 50  0001 C CNN "Vendorpart"
+F 7 "GRM188C80J226ME15D" H 6000 3200 50  0001 C CNN "Mfgrpart"
 	1    6000 3200
 	-1   0    0    1
@@
 F 4 "Murata" H 6300 3200 50  0001 C CNN "Mfgr"
 F 5 "" H 6300 3200 50  0001 C CNN "Part"
-F 6 "490-7196-1-ND" H 6300 3200 50  0001 C CNN "Vendorpart"
-F 7 "GRM188C80G226MEA0D" H 6300 3200 50  0001 C CNN "Mfgrpart"
+F 6 "490-10471-1-ND" H 6300 3200 50  0001 C CNN "Vendorpart"
+F 7 "GRM188C80J226ME15D" H 6300 3200 50  0001 C CNN "Mfgrpart"
 	1    6300 3200
 	-1   0    0    1
@@
 F 4 "Murata" H 6000 3650 50  0001 C CNN "Mfgr"
 F 5 "" H 6000 3650 50  0001 C CNN "Part"
-F 6 "490-7196-1-ND" H 6000 3650 50  0001 C CNN "Vendorpart"
-F 7 "GRM188C80G226MEA0D" H 6000 3650 50  0001 C CNN "Mfgrpart"
+F 6 "490-10471-1-ND" H 6000 3650 50  0001 C CNN "Vendorpart"
+F 7 "GRM188C80J226ME15D" H 6000 3650 50  0001 C CNN "Mfgrpart"
 	1    6000 3650
 	-1   0    0    1
@@
 F 4 "Murata" H 6300 3650 50  0001 C CNN "Mfgr"
 F 5 "" H 6300 3650 50  0001 C CNN "Part"
-F 6 "490-7196-1-ND" H 6300 3650 50  0001 C CNN "Vendorpart"
-F 7 "GRM188C80G226MEA0D" H 6300 3650 50  0001 C CNN "Mfgrpart"
+F 6 "490-10471-1-ND" H 6300 3650 50  0001 C CNN "Vendorpart"
+F 7 "GRM188C80J226ME15D" H 6300 3650 50  0001 C CNN "Mfgrpart"
 	1    6300 3650
 	-1   0    0    1
@@
 F 4 "Murata" H 6000 4100 50  0001 C CNN "Mfgr"
 F 5 "" H 6000 4100 50  0001 C CNN "Part"
-F 6 "490-7196-1-ND" H 6000 4100 50  0001 C CNN "Vendorpart"
-F 7 "GRM188C80G226MEA0D" H 6000 4100 50  0001 C CNN "Mfgrpart"
+F 6 "490-10471-1-ND" H 6000 4100 50  0001 C CNN "Vendorpart"
+F 7 "GRM188C80J226ME15D" H 6000 4100 50  0001 C CNN "Mfgrpart"
 	1    6000 4100
 	-1   0    0    1
@@
 F 4 "Murata" H 6300 4100 50  0001 C CNN "Mfgr"
 F 5 "" H 6300 4100 50  0001 C CNN "Part"
-F 6 "490-7196-1-ND" H 6300 4100 50  0001 C CNN "Vendorpart"
-F 7 "GRM188C80G226MEA0D" H 6300 4100 50  0001 C CNN "Mfgrpart"
+F 6 "490-10471-1-ND" H 6300 4100 50  0001 C CNN "Vendorpart"
+F 7 "GRM188C80J226ME15D" H 6300 4100 50  0001 C CNN "Mfgrpart"
 	1    6300 4100
 	-1   0    0    1
