File: hardware_sbc/SD_MMC.sch (KiCad schematic (older format))
At the start: 14 parts, among them J10 Micro_SD_Card, U1 IMX8MM, U7 SDINBDG4-8G

Commit message: BOM and misc fixes for production of 0.9 boards
Parts:
- C152: Mfgrpart (none) -> GRM155C80J475MEAAD; Part GRM155C80J475MEAAD -> (none)
- C153, C154, C155, C156, C157, C161: Mfgrpart (none) -> GRM033C80J224KE90D; Part GRM033C80J224KE90D -> (none)
- C158: Mfgrpart (none) -> GRM155C80J106ME11D; Part GRM155C80J106ME11D -> (none)
- C159: Mfgrpart (none) -> GRM155C8YA224ME01D; Part GRM155C8YA224ME01D -> (none)
- C160: Mfgrpart (none) -> GRM155C81A105KA12D; Part GRM155C81A105KA12D -> (none)
- J10: Mfgrpart (none) -> 114-00841-68; Part 114-00841-68 -> (none)
- R63: Mfgrpart (none) -> ERJ-2GEJ103X; Part ERJ-2GEJ103X -> (none)
- U1: Mfgrpart (none) -> MIMX8MM6CVTKZAA; Part MIMX8MM6CVTKZAA -> (none)
- U7: Mfgrpart (none) -> SDINBDG4-8G-I1; Part SDINBDG4-8G-I1 -> (none)
Changed lines of the file:
@@
 F 3 "" H 7450 9950 50  0001 C CNN
 F 4 "NXP" H 8200 7200 50  0001 C CNN "Mfgr"
-F 5 "MIMX8MM6CVTKZAA" H 8200 7200 50  0001 C CNN "Part"
+F 5 "" H 8200 7200 50  0001 C CNN "Part"
 F 6 "568-15276-ND" H 8200 7200 50  0001 C CNN "Vendorpart"
+F 7 "MIMX8MM6CVTKZAA" H 8200 7200 50  0001 C CNN "Mfgrpart"
 	9    8200 7200
 	1    0    0    -1
@@
 F 3 "~" H 9700 5900 50  0001 C CNN
 F 4 "Panasonic" H 9700 5900 50  0001 C CNN "Mfgr"
-F 5 "ERJ-2GEJ103X" H 9700 5900 50  0001 C CNN "Part"
+F 5 "" H 9700 5900 50  0001 C CNN "Part"
 F 6 "P10KJCT-ND" H 9700 5900 50  0001 C CNN "Vendorpart"
+F 7 "ERJ-2GEJ103X" H 9700 5900 50  0001 C CNN "Mfgrpart"
 	1    9700 5900
 	1    0    0    -1
@@
 F 3 "~" H 9600 4200 50  0001 C CNN
 F 4 "Murata" H 9600 4200 50  0001 C CNN "Mfgr"
-F 5 "GRM155C8YA224ME01D" H 9600 4200 50  0001 C CNN "Part"
+F 5 "" H 9600 4200 50  0001 C CNN "Part"
 F 6 "490-10446-1-ND" H 9600 4200 50  0001 C CNN "Vendorpart"
+F 7 "GRM155C8YA224ME01D" H 9600 4200 50  0001 C CNN "Mfgrpart"
 	1    9600 4200
 	1    0    0    -1
@@
 F 3 "~" H 5850 4150 50  0001 C CNN
 F 4 "Murata" H 5850 4150 50  0001 C CNN "Mfgr"
-F 5 "GRM033C80J224KE90D" H 5850 4150 50  0001 C CNN "Part"
+F 5 "" H 5850 4150 50  0001 C CNN "Part"
 F 6 "490-10392-1-ND" H 5850 4150 50  0001 C CNN "Vendorpart"
+F 7 "GRM033C80J224KE90D" H 5850 4150 50  0001 C CNN "Mfgrpart"
 	1    5850 4150
 	1    0    0    -1
@@
 F 3 "~" H 6150 4150 50  0001 C CNN
 F 4 "Murata" H 6150 4150 50  0001 C CNN "Mfgr"
-F 5 "GRM033C80J224KE90D" H 6150 4150 50  0001 C CNN "Part"
+F 5 "" H 6150 4150 50  0001 C CNN "Part"
 F 6 "490-10392-1-ND" H 6150 4150 50  0001 C CNN "Vendorpart"
+F 7 "GRM033C80J224KE90D" H 6150 4150 50  0001 C CNN "Mfgrpart"
 	1    6150 4150
 	1    0    0    -1
@@
 F 3 "~" H 6400 4150 50  0001 C CNN
 F 4 "Murata" H 6400 4150 50  0001 C CNN "Mfgr"
-F 5 "GRM033C80J224KE90D" H 6400 4150 50  0001 C CNN "Part"
+F 5 "" H 6400 4150 50  0001 C CNN "Part"
 F 6 "490-10392-1-ND" H 6400 4150 50  0001 C CNN "Vendorpart"
+F 7 "GRM033C80J224KE90D" H 6400 4150 50  0001 C CNN "Mfgrpart"
 	1    6400 4150
 	1    0    0    -1
@@
 F 3 "~" H 6650 4150 50  0001 C CNN
 F 4 "Murata" H 6650 4150 50  0001 C CNN "Mfgr"
-F 5 "GRM155C80J106ME11D" H 6650 4150 50  0001 C CNN "Part"
+F 5 "" H 6650 4150 50  0001 C CNN "Part"
 F 6 "490-13233-1-ND" H 6650 4150 50  0001 C CNN "Vendorpart"
+F 7 "GRM155C80J106ME11D" H 6650 4150 50  0001 C CNN "Mfgrpart"
 	1    6650 4150
 	1    0    0    -1
@@
 F 3 "~" H 4100 4150 50  0001 C CNN
 F 4 "Murata" H 4100 4150 50  0001 C CNN "Mfgr"
-F 5 "GRM033C80J224KE90D" H 4100 4150 50  0001 C CNN "Part"
+F 5 "" H 4100 4150 50  0001 C CNN "Part"
 F 6 "490-10392-1-ND" H 4100 4150 50  0001 C CNN "Vendorpart"
+F 7 "GRM033C80J224KE90D" H 4100 4150 50  0001 C CNN "Mfgrpart"
 	1    4100 4150
 	1    0    0    -1
@@
 F 3 "~" H 3850 4150 50  0001 C CNN
 F 4 "Murata" H 3850 4150 50  0001 C CNN "Mfgr"
-F 5 "GRM033C80J224KE90D" H 3850 4150 50  0001 C CNN "Part"
+F 5 "" H 3850 4150 50  0001 C CNN "Part"
 F 6 "490-10392-1-ND" H 3850 4150 50  0001 C CNN "Vendorpart"
+F 7 "GRM033C80J224KE90D" H 3850 4150 50  0001 C CNN "Mfgrpart"
 	1    3850 4150
 	1    0    0    -1
@@
 F 3 "~" H 3600 4150 50  0001 C CNN
 F 4 "Murata" H 3600 4150 50  0001 C CNN "Mfgr"
-F 5 "GRM155C80J475MEAAD" H 3600 4150 50  0001 C CNN "Part"
+F 5 "" H 3600 4150 50  0001 C CNN "Part"
 F 6 "490-14458-1-ND" H 3600 4150 50  0001 C CNN "Vendorpart"
+F 7 "GRM155C80J475MEAAD" H 3600 4150 50  0001 C CNN "Mfgrpart"
 	1    3600 4150
 	1    0    0    -1
@@
 F 3 "~" H 3650 5150 50  0001 C CNN
 F 4 "Murata" H 3650 5150 50  0001 C CNN "Mfgr"
-F 5 "GRM033C80J224KE90D" H 3650 5150 50  0001 C CNN "Part"
+F 5 "" H 3650 5150 50  0001 C CNN "Part"
 F 6 "490-10392-1-ND" H 3650 5150 50  0001 C CNN "Vendorpart"
+F 7 "GRM033C80J224KE90D" H 3650 5150 50  0001 C CNN "Mfgrpart"
 	1    3650 5150
 	1    0    0    -1
@@
 F 3 "~" H 3400 5150 50  0001 C CNN
 F 4 "Murata" H 3400 5150 50  0001 C CNN "Mfgr"
-F 5 "GRM155C81A105KA12D" H 3400 5150 50  0001 C CNN "Part"
+F 5 "" H 3400 5150 50  0001 C CNN "Part"
 F 6 "490-12699-1-ND" H 3400 5150 50  0001 C CNN "Vendorpart"
+F 7 "GRM155C81A105KA12D" H 3400 5150 50  0001 C CNN "Mfgrpart"
 	1    3400 5150
 	1    0    0    -1
@@
 F 3 "http://katalog.we-online.de/em/datasheet/693072010801.pdf" H 11200 4950 50  0001 C CNN
 F 4 "Amphenol" H 11200 4950 50  0001 C CNN "Mfgr"
-F 5 "114-00841-68" H 11200 4950 50  0001 C CNN "Part"
+F 5 "" H 11200 4950 50  0001 C CNN "Part"
 F 6 "114-00841-68-1-ND" H 11200 4950 50  0001 C CNN "Vendorpart"
+F 7 "114-00841-68" H 11200 4950 50  0001 C CNN "Mfgrpart"
 	1    11200 4950
 	1    0    0    -1
@@
 F 3 "" H 4950 5500 50  0001 L BNN
 F 4 "SanDisk" H 4950 5500 50  0001 C CNN "Mfgr"
-F 5 "SDINBDG4-8G-I1" H 4950 5500 50  0001 C CNN "Part"
+F 5 "" H 4950 5500 50  0001 C CNN "Part"
 F 6 "Mouser" H 4950 5500 50  0001 C CNN "Vendor"
 F 7 "467-SDINBDG4-8G-I1" H 4950 5500 50  0001 C CNN "Vendorpart"
+F 8 "SDINBDG4-8G-I1" H 4950 5500 50  0001 C CNN "Mfgrpart"
 	1    4950 5500
 	1    0    0    -1
