File: hardware_sbc/expansion.sch (KiCad schematic (older format))
At the start: 3 parts, among them J11 DF40HC(3.5)-60DS, J12 DF40HC(3.5)-60DS, U1 IMX8MM

Commit message: BOM and misc fixes for production of 0.9 boards
Parts:
- J11, J12: Mfgrpart (none) -> DF40C-60DP-0.4V(51); Part DF40C-60DP-0.4V(51) -> (none)
- U1: Mfgrpart (none) -> MIMX8MM6CVTKZAA; Part MIMX8MM6CVTKZAA -> (none)
Changed lines of the file:
@@
 F 4 "H11628CT-ND" H 6200 2800 50  0000 C CNN "Vendorpart"
 F 5 "Hirose" H 6200 2800 50  0001 C CNN "Mfgr"
-F 6 "DF40C-60DP-0.4V(51)" H 6200 2800 50  0001 C CNN "Part"
+F 6 "" H 6200 2800 50  0001 C CNN "Part"
+F 7 "DF40C-60DP-0.4V(51)" H 6200 2800 50  0001 C CNN "Mfgrpart"
 	1    6200 2800
 	1    0    0    -1
@@
 F 4 "H11628CT-ND" H 8800 2800 50  0000 C CNN "Vendorpart"
 F 5 "Hirose" H 8800 2800 50  0001 C CNN "Mfgr"
-F 6 "DF40C-60DP-0.4V(51)" H 8800 2800 50  0001 C CNN "Part"
+F 6 "" H 8800 2800 50  0001 C CNN "Part"
+F 7 "DF40C-60DP-0.4V(51)" H 8800 2800 50  0001 C CNN "Mfgrpart"
 	1    8800 2800
 	1    0    0    -1
@@
 F 3 "" H 1300 6350 50  0001 C CNN
 F 4 "NXP" H 2050 3600 50  0001 C CNN "Mfgr"
-F 5 "MIMX8MM6CVTKZAA" H 2050 3600 50  0001 C CNN "Part"
+F 5 "" H 2050 3600 50  0001 C CNN "Part"
 F 6 "568-15276-ND" H 2050 3600 50  0001 C CNN "Vendorpart"
+F 7 "MIMX8MM6CVTKZAA" H 2050 3600 50  0001 C CNN "Mfgrpart"
 	8    2050 3600
 	1    0    0    -1
@@
 F 3 "" H 3500 7400 50  0001 C CNN
 F 4 "NXP" H 4300 4650 50  0001 C CNN "Mfgr"
-F 5 "MIMX8MM6CVTKZAA" H 4300 4650 50  0001 C CNN "Part"
+F 5 "" H 4300 4650 50  0001 C CNN "Part"
 F 6 "568-15276-ND" H 4300 4650 50  0001 C CNN "Vendorpart"
+F 7 "MIMX8MM6CVTKZAA" H 4300 4650 50  0001 C CNN "Mfgrpart"
 	10   4300 4650
 	1    0    0    1
@@
 F 3 "" H 900 11250 50  0001 C CNN
 F 4 "NXP" H 1650 8500 50  0001 C CNN "Mfgr"
-F 5 "MIMX8MM6CVTKZAA" H 1650 8500 50  0001 C CNN "Part"
+F 5 "" H 1650 8500 50  0001 C CNN "Part"
 F 6 "568-15276-ND" H 1650 8500 50  0001 C CNN "Vendorpart"
+F 7 "MIMX8MM6CVTKZAA" H 1650 8500 50  0001 C CNN "Mfgrpart"
 	4    1650 8500
 	1    0    0    -1
@@
 F 3 "" H 900 9050 50  0001 C CNN
 F 4 "NXP" H 1650 6300 50  0001 C CNN "Mfgr"
-F 5 "MIMX8MM6CVTKZAA" H 1650 6300 50  0001 C CNN "Part"
+F 5 "" H 1650 6300 50  0001 C CNN "Part"
 F 6 "568-15276-ND" H 1650 6300 50  0001 C CNN "Vendorpart"
+F 7 "MIMX8MM6CVTKZAA" H 1650 6300 50  0001 C CNN "Mfgrpart"
 	5    1650 6300
 	1    0    0    -1
