File: hardware_sbc/CPU-power.kicad_sch (KiCad schematic)
At the start: 57 parts, among them U1 IMX8MM

Commit message: Updated production files and fixed schematic link issue.
Fixed schematic unit number issue and re-linked to PCB.
New gerbers, STEP file, schematic PDF.
Deleted old KiCAD 6 files.
Parts:
- renumbered U1 to U?
Changed lines of the file:
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@@
 		(on_board yes)
 		(dnp no)
-		(property "Reference" "#PWR075"
+		(property "Reference" "#PWR?"
 			(at 297.18 195.58 0)
 			(effects
@@
 		(on_board yes)
 		(dnp no)
-		(property "Reference" "#PWR077"
+		(property "Reference" "#PWR?"
 			(at 359.41 203.2 0)
 			(effects
@@
 		(on_board yes)
 		(dnp no)
-		(property "Reference" "U1"
+		(property "Reference" "U?"
 			(at 328.295 52.705 0)
 			(effects
@@
 		(on_board yes)
 		(dnp no)
-		(property "Reference" "U1"
+		(property "Reference" "U?"
 			(at 125.095 32.639 0)
 			(effects
