File: hardware_sbc/PCIe.kicad_sch (KiCad schematic)
At the start: 23 parts, among them J5 Bus_PCI_Express_Mini, U13 MIC94164, U1C IMX8MM

Commit message: Updated production files and fixed schematic link issue.
Fixed schematic unit number issue and re-linked to PCB.
New gerbers, STEP file, schematic PDF.
Deleted old KiCAD 6 files.
Parts:
- renumbered C130 to C?, C131 to C?, C124 to C?, J5 to J?, U1C to U1
Connections:
- net PCIE_CLK_N: now also U1.A21 (PCIE_CLK_N)
- net PCIE_CLK_P: now also U1.B21 (PCIE_CLK_P)
- net PCIE_RXN_N: now also U1.A19 (PCIE_RXN_N)
- net PCIE_RXN_P: now also U1.B19 (PCIE_RXN_P)
- net PCIE_TXN_1_N: now also U1.A20 (PCIE_TXN_N)
- net PCIE_TXN_1_P: now also U1.B20 (PCIE_TXN_P)
- net at R36.1: now also U1.D19 (PCIE_RESREF)
Changed lines of the file:
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@@
 	(label "PCIE_CLK_P"
 		(at 152.4 92.71 0)
+		(fields_autoplaced yes)
 		(effects
 			(font
@@
 	(label "PCIE_RXN_P"
 		(at 152.4 100.33 0)
+		(fields_autoplaced yes)
 		(effects
 			(font
@@
 	(label "PCIE_RXN_N"
 		(at 152.4 97.79 0)
+		(fields_autoplaced yes)
 		(effects
 			(font
@@
 	(label "PCIE_CLK_N"
 		(at 152.4 90.17 0)
+		(fields_autoplaced yes)
 		(effects
 			(font
@@
 	(label "PCIE_TXN_P"
 		(at 152.4 105.41 0)
+		(fields_autoplaced yes)
 		(effects
 			(font
@@
 	(label "PCIE_TXN_1_P"
 		(at 125.73 107.95 0)
+		(fields_autoplaced yes)
 		(effects
 			(font
@@
 	(label "PCIE_TXN_N"
 		(at 152.4 102.87 0)
+		(fields_autoplaced yes)
 		(effects
 			(font
@@
 	(label "PCIE_TXN_1_N"
 		(at 125.73 105.41 0)
+		(fields_autoplaced yes)
 		(effects
 			(font
@@
 		(shape input)
 		(at 133.35 72.39 180)
+		(fields_autoplaced yes)
 		(effects
 			(font
@@
 		(shape input)
 		(at 35.56 52.07 180)
+		(fields_autoplaced yes)
 		(effects
 			(font
@@
 		(shape input)
 		(at 133.35 69.85 180)
+		(fields_autoplaced yes)
 		(effects
 			(font
@@
 		(shape input)
 		(at 160.02 60.96 90)
+		(fields_autoplaced yes)
 		(effects
 			(font
@@
 		(shape input)
 		(at 162.56 60.96 90)
+		(fields_autoplaced yes)
 		(effects
 			(font
@@
 		(on_board yes)
 		(dnp no)
-		(property "Reference" "J5"
+		(property "Reference" "J?"
 			(at 185.5216 63.6524 90)
 			(effects
@@
 		(lib_id "mxenc:MIMX8MM6DVTLZAA")
 		(at 93.98 156.21 0)
-		(unit 1)
+		(unit 3)
 		(exclude_from_sim no)
 		(in_bom yes)
 		(on_board yes)
 		(dnp no)
-		(property "Reference" "U1C"
+		(property "Reference" "U1"
 			(at 96.7232 83.439 0)
 			(effects
@@
 			(project "kimchi_micro"
 				(path "/394ea9d6-84ac-414f-b42c-59edf258c746/00000000-0000-0000-0000-00005d31363c"
-					(reference "U1C")
-					(unit 1)
+					(reference "U1")
+					(unit 3)
 				)
 			)
@@
 		(on_board yes)
 		(dnp no)
-		(property "Reference" "C130"
+		(property "Reference" "C?"
 			(at 200.66 133.35 0)
 			(effects
@@
 		(on_board yes)
 		(dnp no)
-		(property "Reference" "C131"
+		(property "Reference" "C?"
 			(at 207.01 133.35 0)
 			(effects
@@
 		(on_board yes)
 		(dnp no)
-		(property "Reference" "C124"
+		(property "Reference" "C?"
 			(at 139.7 133.35 0)
 			(effects
