File: hardware_sbc/PMIC.kicad_sch (KiCad schematic)
At the start: 60 parts, among them U4 BD71847MWV, Y2 Crystal

Commit message: Updated production files and fixed schematic link issue.
Fixed schematic unit number issue and re-linked to PCB.
New gerbers, STEP file, schematic PDF.
Deleted old KiCAD 6 files.
Parts:
- renumbered U4 to U?
Changed lines of the file:
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@@
 		(shape input)
 		(at 96.52 184.15 180)
+		(fields_autoplaced yes)
 		(effects
 			(font
@@
 		(shape output)
 		(at 179.07 175.26 0)
+		(fields_autoplaced yes)
 		(effects
 			(font
@@
 		(shape input)
 		(at 308.61 93.98 180)
+		(fields_autoplaced yes)
 		(effects
 			(font
@@
 		(shape input)
 		(at 96.52 173.99 180)
+		(fields_autoplaced yes)
 		(effects
 			(font
@@
 		(shape bidirectional)
 		(at 96.52 163.83 180)
+		(fields_autoplaced yes)
 		(effects
 			(font
@@
 		(shape output)
 		(at 179.07 168.91 0)
+		(fields_autoplaced yes)
 		(effects
 			(font
@@
 		(shape output)
 		(at 179.07 187.96 0)
+		(fields_autoplaced yes)
 		(effects
 			(font
@@
 		(shape output)
 		(at 179.07 181.61 0)
+		(fields_autoplaced yes)
 		(effects
 			(font
@@
 		(shape input)
 		(at 96.52 179.07 180)
+		(fields_autoplaced yes)
 		(effects
 			(font
@@
 		(shape input)
 		(at 96.52 168.91 180)
+		(fields_autoplaced yes)
 		(effects
 			(font
@@
 		(shape input)
 		(at 96.52 161.29 180)
+		(fields_autoplaced yes)
 		(effects
 			(font
@@
 		(on_board yes)
 		(dnp no)
-		(property "Reference" "U4"
+		(property "Reference" "U?"
 			(at 106.045 36.3982 0)
 			(effects
@@
 		(on_board yes)
 		(dnp no)
-		(property "Reference" "U4"
+		(property "Reference" "U?"
 			(at 330.2 33.8582 0)
 			(effects
@@
 		(on_board yes)
 		(dnp no)
-		(property "Reference" "U4"
+		(property "Reference" "U?"
 			(at 141.605 136.3726 0)
 			(effects
